File: Hardware/PCB/dualvca/dualvca.kicad_pcb (KiCad board)
At the start: 2 copper layers, 183 x 155 mm, 93 parts, among them J1 AudioJack2, J101 Conn_01x15, J102 Conn_01x15, J103 Synth_power_2x5, J2 AudioJack2, J3 AudioJack2, J4 AudioJack2, J5 AudioJack2, J6 AudioJack2, J7 AudioJack2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

Commit message: KiCad 7, libraries to folder
Parts:
- renumbered TP1 to TP101, TP2 to TP102, TP3 to TP103, TP4 to TP104, TP5 to TP105, TP6 to TP106
Changed lines of the file:
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@@
     (property "ki_keywords" "test point tp")
     (attr exclude_from_pos_files exclude_from_bom)
-    (fp_text reference "TP2" (at 0 -3.048 90) (layer "F.SilkS")
+    (fp_text reference "TP102" (at 0 -3.048 90) (layer "F.SilkS")
         (effects (font (size 0.75 0.75) (thickness 0.15)))
     )
@@
     (property "ki_keywords" "test point tp")
     (attr exclude_from_pos_files exclude_from_bom)
-    (fp_text reference "TP6" (at 0 -3.048 90) (layer "F.SilkS")
+    (fp_text reference "TP106" (at 0 -3.048 90) (layer "F.SilkS")
         (effects (font (size 0.75 0.75) (thickness 0.15)))
     )
@@
     (property "ki_keywords" "test point tp")
     (attr exclude_from_pos_files exclude_from_bom)
-    (fp_text reference "TP4" (at 0 -3.048 90) (layer "F.SilkS")
+    (fp_text reference "TP104" (at 0 -3.048 90) (layer "F.SilkS")
         (effects (font (size 0.75 0.75) (thickness 0.15)))
     )
@@
     (property "ki_keywords" "test point tp")
     (attr exclude_from_pos_files exclude_from_bom)
-    (fp_text reference "TP5" (at 0 -3.048 90) (layer "F.SilkS")
+    (fp_text reference "TP105" (at 0 -3.048 90) (layer "F.SilkS")
         (effects (font (size 0.75 0.75) (thickness 0.15)))
     )
@@
     (property "ki_keywords" "test point tp")
     (attr exclude_from_pos_files exclude_from_bom)
-    (fp_text reference "TP1" (at 0 -3.048 90) (layer "F.SilkS")
+    (fp_text reference "TP101" (at 0 -3.048 90) (layer "F.SilkS")
         (effects (font (size 0.75 0.75) (thickness 0.15)))
     )
@@
     (property "ki_keywords" "test point tp")
     (attr exclude_from_pos_files exclude_from_bom)
-    (fp_text reference "TP3" (at 0 -3.048 90) (layer "F.SilkS")
+    (fp_text reference "TP103" (at 0 -3.048 90) (layer "F.SilkS")
         (effects (font (size 0.75 0.75) (thickness 0.15)))
     )
