File: Hardware/PCB/dualvca/potsw.kicad_sch (KiCad schematic)
At the start: 15 parts, among them SW1 SW_SPDT, SW2 SW_SPDT

Commit message: KiCad 7, libraries to folder
Parts:
- renumbered TP7 to TP1, TP8 to TP2, TP9 to TP3
Changed lines of the file:
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@@
   (symbol (lib_id "AO_symbols:TestPoint") (at 220.98 128.27 0) (mirror x) (unit 1)
     (in_bom no) (on_board yes) (dnp no) (fields_autoplaced)
-    (property "Reference" "TP7" (at 218.44 130.937 0)
+    (property "Reference" "TP1" (at 218.44 130.937 0)
       (effects (font (size 1.27 1.27)) (justify right))
     )
@@
         )
         (path "/1fce46f5-2003-4c7e-915f-b9b7dfc679d7/154653f8-fa65-4bcf-b100-6b1eefd55b94"
-          (reference "TP4") (unit 1)
+          (reference "TP104") (unit 1)
         )
       )
@@
   (symbol (lib_id "AO_symbols:TestPoint") (at 232.41 129.54 0) (unit 1)
     (in_bom no) (on_board yes) (dnp no) (fields_autoplaced)
-    (property "Reference" "TP8" (at 234.95 125.603 0)
+    (property "Reference" "TP2" (at 234.95 125.603 0)
       (effects (font (size 1.27 1.27)) (justify left))
     )
@@
         )
         (path "/1fce46f5-2003-4c7e-915f-b9b7dfc679d7/154653f8-fa65-4bcf-b100-6b1eefd55b94"
-          (reference "TP5") (unit 1)
+          (reference "TP105") (unit 1)
         )
       )
@@
   (symbol (lib_id "AO_symbols:TestPoint") (at 246.38 129.54 0) (unit 1)
     (in_bom no) (on_board yes) (dnp no) (fields_autoplaced)
-    (property "Reference" "TP9" (at 248.92 125.603 0)
+    (property "Reference" "TP3" (at 248.92 125.603 0)
       (effects (font (size 1.27 1.27)) (justify left))
     )
@@
         )
         (path "/1fce46f5-2003-4c7e-915f-b9b7dfc679d7/154653f8-fa65-4bcf-b100-6b1eefd55b94"
-          (reference "TP6") (unit 1)
-        )
-      )
+          (reference "TP106") (unit 1)
+        )
+      )
