File: Hardware/PCB/dualvca/potsw.kicad_sch (KiCad schematic)
At the start: 15 parts, among them SW1 SW_SPDT, SW2 SW_SPDT

Commit message: Hardware, BOM
Parts:
- added ZKN101, ZKN102, ZKN103, ZKN104: Knob_MF-A03, symbol AO_symbols:Knob
Other:
- note added: "Hardware"
