File: Hardware/PCB/dualvca/main.kicad_sch (KiCad schematic)
At the start: 76 parts, among them J1 AudioJack2, J103 Synth_power_2x5, J2 AudioJack2, J3 AudioJack2, J4 AudioJack2, J5 AudioJack2, J6 AudioJack2, J7 AudioJack2, J8 AudioJack2_SwitchT, Q1 2N3904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

Commit message: KiCad 7, libraries to folder
Parts:
- renumbered TP7 to TP101, TP8 to TP102, TP9 to TP103
Changed lines of the file:
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@@
   (symbol (lib_id "AO_symbols:TestPoint") (at 114.3 153.67 0) (mirror x) (unit 1)
     (in_bom no) (on_board yes) (dnp no) (fields_autoplaced)
-    (property "Reference" "TP7" (at 111.76 156.337 0)
+    (property "Reference" "TP101" (at 111.76 156.337 0)
       (effects (font (size 1.27 1.27)) (justify right))
     )
@@
       (project "dualvca"
         (path "/1fce46f5-2003-4c7e-915f-b9b7dfc679d7/f38c5955-04d6-42ca-a935-84c438c12043"
-          (reference "TP1") (unit 1)
+          (reference "TP101") (unit 1)
         )
       )
@@
   (symbol (lib_id "AO_symbols:TestPoint") (at 139.7 154.94 0) (unit 1)
     (in_bom no) (on_board yes) (dnp no) (fields_autoplaced)
-    (property "Reference" "TP9" (at 142.24 151.003 0)
+    (property "Reference" "TP103" (at 142.24 151.003 0)
       (effects (font (size 1.27 1.27)) (justify left))
     )
@@
       (project "dualvca"
         (path "/1fce46f5-2003-4c7e-915f-b9b7dfc679d7/f38c5955-04d6-42ca-a935-84c438c12043"
-          (reference "TP3") (unit 1)
+          (reference "TP103") (unit 1)
         )
       )
@@
   (symbol (lib_id "AO_symbols:TestPoint") (at 125.73 154.94 0) (unit 1)
     (in_bom no) (on_board yes) (dnp no) (fields_autoplaced)
-    (property "Reference" "TP8" (at 128.27 151.003 0)
+    (property "Reference" "TP102" (at 128.27 151.003 0)
       (effects (font (size 1.27 1.27)) (justify left))
     )
@@
       (project "dualvca"
         (path "/1fce46f5-2003-4c7e-915f-b9b7dfc679d7/f38c5955-04d6-42ca-a935-84c438c12043"
-          (reference "TP2") (unit 1)
-        )
-      )
+          (reference "TP102") (unit 1)
+        )
+      )

Commit message: Hardware, BOM
Parts:
- added J104: DIP-14, symbol AO_symbols:DIP-14
- added J105: DIP-16, symbol AO_symbols:DIP-16
- RV18, RV41, RV45, RV47: Manufacturer (none) -> Bourns; Part (none) -> 3296W
Other:
- note added: "Hardware"
