File: Hardware/Panel/mfos_vca-panel/mfos_vca-panel.kicad_pcb (KiCad board)
At the start: 2 copper layers, 100 x 200 mm, 18 parts

Commit message: gerbers
Parts:
- H1, H10, H12, H6: footprint Kosmo_panel_NPTH:Kosmo_Pot_Hole -> Kosmo_panel:Kosmo_Pot_Hole
- H11, H13, H14, H15, H16, H3, H5, H9: footprint Kosmo_panel_NPTH:Kosmo_Jack_Hole -> Kosmo_panel:Kosmo_Jack_Hole
- H2, H7: footprint Kosmo_panel_NPTH:Kosmo_Switch_Hole -> Kosmo_panel:Kosmo_Switch_Hole
- H4, H8: footprint Kosmo_panel_NPTH:Kosmo_Panel_Dual_Slotted_Mounting_Holes -> Kosmo_panel:Kosmo_Panel_Dual_Slotted_Mounting_Holes
