File: Hardware/Panel/mfos_vca-panel/mfos_vca-panel.kicad_sch (KiCad schematic)
At the start: 18 parts

Commit message: gerbers
Parts:
- H1, H10, H12, H6: footprint Kosmo_panel_NPTH:Kosmo_Pot_Hole -> Kosmo_panel:Kosmo_Pot_Hole
- H11, H13, H14, H15, H16, H3, H5, H9: footprint Kosmo_panel_NPTH:Kosmo_Jack_Hole -> Kosmo_panel:Kosmo_Jack_Hole
- H2, H7: footprint Kosmo_panel_NPTH:Kosmo_Switch_Hole -> Kosmo_panel:Kosmo_Switch_Hole
- H4, H8: footprint Kosmo_panel_NPTH:Kosmo_Panel_Dual_Slotted_Mounting_Holes -> Kosmo_panel:Kosmo_Panel_Dual_Slotted_Mounting_Holes
Changed lines of the file:
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@@
+    )
+  )
+  (symbol (lib_id "power:PWR_FLAG") (at 229.87 74.93 0) (unit 1)
+    (in_bom yes) (on_board yes) (dnp no) (fields_autoplaced)
+    (property "Reference" "#FLG01" (at 229.87 73.025 0)
+      (effects (font (size 1.27 1.27)) hide)
+    )
+    (property "Value" "PWR_FLAG" (at 229.87 71.12 0)
+      (effects (font (size 1.27 1.27)))
+    )
+    (property "Footprint" "" (at 229.87 74.93 0)
+      (effects (font (size 1.27 1.27)) hide)
+    )
+    (property "Datasheet" "~" (at 229.87 74.93 0)
+      (effects (font (size 1.27 1.27)) hide)
+    )
+    (pin "1")
+    (instances
+      (project "mfos_vca-panel"
+        (path "/23a7ac9b-26cd-4330-94ee-51b93744d635"
+          (reference "#FLG01") (unit 1)
+        )
+      )
     )
   )
@@
       (effects (font (size 1.27 1.27)) (justify left))
     )
-    (property "Footprint" "Kosmo_panel_NPTH:Kosmo_Jack_Hole" (at 168.91 81.28 0)
+    (property "Footprint" "Kosmo_panel:Kosmo_Jack_Hole" (at 168.91 81.28 0)
       (effects (font (size 1.27 1.27)) hide)
     )
@@
       (effects (font (size 1.27 1.27)) (justify left))
     )
-    (property "Footprint" "Kosmo_panel_NPTH:Kosmo_Jack_Hole" (at 86.36 81.28 0)
+    (property "Footprint" "Kosmo_panel:Kosmo_Jack_Hole" (at 86.36 81.28 0)
       (effects (font (size 1.27 1.27)) hide)
     )
@@
       (effects (font (size 1.27 1.27)) (justify left))
     )
-    (property "Footprint" "Kosmo_panel_NPTH:Kosmo_Jack_Hole" (at 102.87 81.28 0)
+    (property "Footprint" "Kosmo_panel:Kosmo_Jack_Hole" (at 102.87 81.28 0)
       (effects (font (size 1.27 1.27)) hide)
     )
@@
       (effects (font (size 1.27 1.27)) (justify left))
     )
-    (property "Footprint" "Kosmo_panel_NPTH:Kosmo_Pot_Hole" (at 139.7 53.34 0)
+    (property "Footprint" "Kosmo_panel:Kosmo_Pot_Hole" (at 139.7 53.34 0)
       (effects (font (size 1.27 1.27)) hide)
     )
@@
       (effects (font (size 1.27 1.27)) (justify left))
     )
-    (property "Footprint" "Kosmo_panel_NPTH:Kosmo_Jack_Hole" (at 135.89 81.28 0)
+    (property "Footprint" "Kosmo_panel:Kosmo_Jack_Hole" (at 135.89 81.28 0)
       (effects (font (size 1.27 1.27)) hide)
     )
@@
       (effects (font (size 1.27 1.27)) (justify left))
     )
-    (property "Footprint" "Kosmo_panel_NPTH:Kosmo_Switch_Hole" (at 108.585 64.516 0)
+    (property "Footprint" "Kosmo_panel:Kosmo_Switch_Hole" (at 108.585 64.516 0)
       (effects (font (size 1.27 1.27)) hide)
     )
@@
       (effects (font (size 1.27 1.27)) (justify left))
     )
-    (property "Footprint" "Kosmo_panel_NPTH:Kosmo_Jack_Hole" (at 152.4 81.28 0)
+    (property "Footprint" "Kosmo_panel:Kosmo_Jack_Hole" (at 152.4 81.28 0)
       (effects (font (size 1.27 1.27)) hide)
     )
@@
     )
   )
+  (symbol (lib_id "power:GND") (at 229.87 74.93 0) (unit 1)
+    (in_bom yes) (on_board yes) (dnp no)
+    (property "Reference" "#PWR02" (at 229.87 81.28 0)
+      (effects (font (size 1.27 1.27)) hide)
+    )
+    (property "Value" "GND" (at 229.997 79.3242 0)
+      (effects (font (size 1.27 1.27)))
+    )
+    (property "Footprint" "" (at 229.87 74.93 0)
+      (effects (font (size 1.27 1.27)) hide)
+    )
+    (property "Datasheet" "" (at 229.87 74.93 0)
+      (effects (font (size 1.27 1.27)) hide)
+    )
+    (pin "1")
+    (instances
+      (project "mfos_vca-panel"
+        (path "/23a7ac9b-26cd-4330-94ee-51b93744d635"
+          (reference "#PWR02") (unit 1)
+        )
+      )
+    )
+  )
   (symbol (lib_id "Kosmo:Mounting_Holes_Slotted") (at 86.36 102.87 0) (unit 1)
     (in_bom yes) (on_board yes) (dnp no) (fields_autoplaced)
@@
       (effects (font (size 1.27 1.27)) (justify left))
     )
-    (property "Footprint" "Kosmo_panel_NPTH:Kosmo_Panel_Dual_Slotted_Mounting_Holes" (at 86.36 102.87 0)
+    (property "Footprint" "Kosmo_panel:Kosmo_Panel_Dual_Slotted_Mounting_Holes" (at 86.36 102.87 0)
       (effects (font (size 1.27 1.27)) hide)
     )
@@
       (effects (font (size 1.27 1.27)) (justify left))
     )
-    (property "Footprint" "Kosmo_panel_NPTH:Kosmo_Jack_Hole" (at 119.38 81.28 0)
+    (property "Footprint" "Kosmo_panel:Kosmo_Jack_Hole" (at 119.38 81.28 0)
       (effects (font (size 1.27 1.27)) hide)
     )
@@
       (effects (font (size 1.27 1.27)) (justify left))
     )
-    (property "Footprint" "Kosmo_panel_NPTH:Kosmo_Pot_Hole" (at 121.92 53.34 0)
+    (property "Footprint" "Kosmo_panel:Kosmo_Pot_Hole" (at 121.92 53.34 0)
       (effects (font (size 1.27 1.27)) hide)
     )
@@
       (effects (font (size 1.27 1.27)) (justify left))
     )
-    (property "Footprint" "Kosmo_panel_NPTH:Kosmo_Switch_Hole" (at 86.995 64.516 0)
+    (property "Footprint" "Kosmo_panel:Kosmo_Switch_Hole" (at 86.995 64.516 0)
       (effects (font (size 1.27 1.27)) hide)
     )
@@
       (effects (font (size 1.27 1.27)) (justify left))
     )
-    (property "Footprint" "Kosmo_panel_NPTH:Kosmo_Jack_Hole" (at 185.42 81.28 0)
+    (property "Footprint" "Kosmo_panel:Kosmo_Jack_Hole" (at 185.42 81.28 0)
       (effects (font (size 1.27 1.27)) hide)
     )
@@
       (effects (font (size 1.27 1.27)) (justify left))
     )
-    (property "Footprint" "Kosmo_panel_NPTH:Kosmo_Pot_Hole" (at 104.14 53.34 0)
+    (property "Footprint" "Kosmo_panel:Kosmo_Pot_Hole" (at 104.14 53.34 0)
       (effects (font (size 1.27 1.27)) hide)
     )
@@
       (effects (font (size 1.27 1.27)) (justify left))
     )
-    (property "Footprint" "Kosmo_panel_NPTH:Kosmo_Pot_Hole" (at 86.36 53.34 0)
+    (property "Footprint" "Kosmo_panel:Kosmo_Pot_Hole" (at 86.36 53.34 0)
       (effects (font (size 1.27 1.27)) hide)
     )
@@
       (effects (font (size 1.27 1.27)) (justify left))
     )
-    (property "Footprint" "Kosmo_panel_NPTH:Kosmo_Panel_Dual_Slotted_Mounting_Holes" (at 114.3 102.87 0)
+    (property "Footprint" "Kosmo_panel:Kosmo_Panel_Dual_Slotted_Mounting_Holes" (at 114.3 102.87 0)
       (effects (font (size 1.27 1.27)) hide)
     )
@@
       (effects (font (size 1.27 1.27)) (justify left))
     )
-    (property "Footprint" "Kosmo_panel_NPTH:Kosmo_Jack_Hole" (at 201.93 81.28 0)
-      (effects (font (size 1.27 1.27)) hide)
-    )
+    (property "Footprint" "Kosmo_panel:Kosmo_Jack_Hole" (at 201.93 81.28 0)
+      (effects (font (size 1.27 1.27)) hide)
+    )
