File: Hardware/dualvca/main.kicad_sch (KiCad schematic)
At the start: 78 parts, among them J1 AudioJack2, J103 Synth_power_2x5, J104 DIP-14, J105 DIP-16, J2 AudioJack2, J3 AudioJack2, J4 AudioJack2, J5 AudioJack2, J6 AudioJack2, J7 AudioJack2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

Commit message: Docs
Parts:
- B101, GRAF101, GRAF103, GRAF104: now left out of the parts list
Changed lines of the file:
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@@
   )
   (symbol (lib_id "AO_symbols:Graphic") (at 66.04 142.24 0) (unit 1)
-    (in_bom yes) (on_board yes) (dnp no) (fields_autoplaced)
+    (in_bom no) (on_board yes) (dnp no) (fields_autoplaced)
     (property "Reference" "GRAF101" (at 73.025 141.3315 0)
       (effects (font (size 1.27 1.27)) (justify left))
@@
   )
   (symbol (lib_id "AO_symbols:Board") (at 68.58 163.83 0) (unit 1)
-    (in_bom yes) (on_board yes) (dnp no) (fields_autoplaced)
+    (in_bom no) (on_board yes) (dnp no) (fields_autoplaced)
     (property "Reference" "B101" (at 74.295 162.9215 0)
       (effects (font (size 1.27 1.27)) (justify left))
@@
   )
   (symbol (lib_id "AO_symbols:Graphic") (at 66.04 149.86 0) (unit 1)
-    (in_bom yes) (on_board yes) (dnp no) (fields_autoplaced)
+    (in_bom no) (on_board yes) (dnp no) (fields_autoplaced)
     (property "Reference" "GRAF103" (at 73.66 149.225 0)
       (effects (font (size 1.27 1.27)) (justify left))
@@
   )
   (symbol (lib_id "AO_symbols:Graphic") (at 66.04 157.48 0) (unit 1)
-    (in_bom yes) (on_board yes) (dnp no) (fields_autoplaced)
+    (in_bom no) (on_board yes) (dnp no) (fields_autoplaced)
     (property "Reference" "GRAF104" (at 73.66 156.845 0)
       (effects (font (size 1.27 1.27)) (justify left))
