File: Hardware/dualvca/potsw.kicad_sch (KiCad schematic)
At the start: 19 parts, among them SW1 SW_SPDT, SW2 SW_SPDT

Commit message: Docs
Parts:
- B102, GRAF102: now left out of the parts list
Changed lines of the file:
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@@
   )
   (symbol (lib_id "AO_symbols:Board") (at 68.58 187.96 0) (unit 1)
-    (in_bom yes) (on_board yes) (dnp no) (fields_autoplaced)
+    (in_bom no) (on_board yes) (dnp no) (fields_autoplaced)
     (property "Reference" "B102" (at 74.295 187.0515 0)
       (effects (font (size 1.27 1.27)) (justify left))
@@
   )
   (symbol (lib_id "AO_symbols:Graphic") (at 67.31 165.1 0) (unit 1)
-    (in_bom yes) (on_board yes) (dnp no) (fields_autoplaced)
+    (in_bom no) (on_board yes) (dnp no) (fields_autoplaced)
     (property "Reference" "GRAF102" (at 74.295 164.1915 0)
       (effects (font (size 1.27 1.27)) (justify left))
